File: pcb/labio-imu.sch (KiCad schematic (older format))
At the start: 8 parts

Commit message: finish rpi to module connections
* use dip switches to disable/configure blocks
* add light sensor
* fix motor controller sense resistors
* fix overused jtag probe pins
Parts:
- added SW?: DIP_SWITCH_X04, symbol DIP_SWITCH_X04
Connections:
- net labels added: INT, INT_J, SCL_J, SDA_J, VDD3V3_J
- net labels removed: INT_MAG, INT_XL
- wire segments 34 -> 55
Changed lines of the file:
@@
 $Descr A4 11693 8268
 encoding utf-8
-Sheet 6 7
+Sheet 5 7
 Title ""
 Date ""
@@
 	1    0    0    -1
 $EndComp
-Text HLabel 3400 2300 0    60   Input ~ 0
-VDD3V3
 $Comp
 L GND #PWR?
@@
 	3400 3000 3400 2900
 Wire Wire Line
-	3400 2900 5100 2900
+	3400 2900 3500 2900
+Wire Wire Line
+	3500 2900 3900 2900
+Wire Wire Line
+	3900 2900 4300 2900
+Wire Wire Line
+	4300 2900 4700 2900
+Wire Wire Line
+	4700 2900 5000 2900
+Wire Wire Line
+	5000 2900 5100 2900
 Wire Wire Line
 	5100 2800 5000 2800
@@
 Connection ~ 3500 2900
 Wire Wire Line
-	3400 2300 5100 2300
+	2800 2300 3500 2300
+Wire Wire Line
+	3500 2300 3900 2300
+Wire Wire Line
+	3900 2300 4300 2300
+Wire Wire Line
+	4300 2300 5100 2300
 Wire Wire Line
 	3500 2300 3500 2600
@@
 Connection ~ 3900 2300
 Wire Wire Line
-	4300 2300 4300 2600
+	4300 2300 4300 2400
+Wire Wire Line
+	4300 2400 4300 2600
 Connection ~ 4300 2300
 Wire Wire Line
@@
 Connection ~ 4300 2400
 NoConn ~ 6500 2900
-Text HLabel 6900 2800 2    60   Input ~ 0
-INT_XL
-Wire Wire Line
-	6900 2800 6500 2800
-Text HLabel 6900 2700 2    60   Input ~ 0
-INT_MAG
-Wire Wire Line
-	6900 2700 6500 2700
-Text HLabel 6900 2500 2    60   Input ~ 0
+Text HLabel 7700 2700 2    60   Input ~ 0
+INT
+Wire Wire Line
+	7100 2700 6600 2700
+Wire Wire Line
+	6600 2700 6500 2700
+Text HLabel 7700 2500 2    60   Input ~ 0
 SCL
-Text HLabel 6900 2600 2    60   Input ~ 0
+Text HLabel 7700 2600 2    60   Input ~ 0
 SDA
-Text HLabel 6900 2300 2    60   Input ~ 0
+Text HLabel 7700 2400 2    60   Input ~ 0
 VDD3V3
 Wire Wire Line
-	6900 2600 6500 2600
-Wire Wire Line
-	6500 2500 6900 2500
-Wire Wire Line
-	6900 2300 6500 2300
+	7100 2600 6500 2600
+Wire Wire Line
+	6500 2500 7100 2500
 Wire Wire Line
 	6500 2400 6600 2400
 Wire Wire Line
-	6600 2400 6600 2300
-Connection ~ 6600 2300
+	6600 2400 7100 2400
 $Comp
 L BMP180 U?
@@
 	1    0    0    -1
 $EndComp
-Text HLabel 4400 4500 0    60   Input ~ 0
-VDD3V3
 $Comp
 L C_Small C?
@@
 $EndComp
 Wire Wire Line
-	4400 4500 5300 4500
+	3800 4500 4500 4500
+Wire Wire Line
+	4500 4500 4900 4500
+Wire Wire Line
+	4900 4500 5300 4500
 Wire Wire Line
 	4500 4700 4500 4500
 Connection ~ 4500 4500
 Wire Wire Line
-	4900 4700 4900 4500
+	4900 4700 4900 4600
+Wire Wire Line
+	4900 4600 4900 4500
 Connection ~ 4900 4500
 Wire Wire Line
@@
 	5200 4800 5200 5000
 Wire Wire Line
-	5200 5000 4400 5000
+	5200 5000 4900 5000
+Wire Wire Line
+	4900 5000 4500 5000
+Wire Wire Line
+	4500 5000 4400 5000
 Wire Wire Line
 	4400 5000 4400 5100
@@
 	1    0    0    -1
 $EndComp
-Text HLabel 6900 4600 2    60   Input ~ 0
-SCL
-Text HLabel 6900 4700 2    60   Input ~ 0
-SDA
 Wire Wire Line
 	6900 4600 6300 4600
@@
 Text Notes 4400 4400 0    60   ~ 0
 1mA max
+Wire Wire Line
+	6500 2800 6600 2800
+Wire Wire Line
+	6600 2800 6600 2700
+Connection ~ 6600 2700
+$Comp
+L DIP_SWITCH_X04 SW?
+U 1 1 576D37BB
+P 7350 2550
+F 0 "SW?" H 7350 2800 50  0000 C CNN
+F 1 "DIP_SWITCH_X04" H 7350 2300 50  0000 C CNN
+F 2 "" H 7350 1350 50  0000 C CNN
+F 3 "" H 7350 1350 50  0000 C CNN
+	1    7350 2550
+	1    0    0    -1
+$EndComp
+Wire Wire Line
+	6600 2400 6600 2300
+Wire Wire Line
+	6600 2300 6500 2300
+Connection ~ 6600 2400
+Wire Wire Line
+	7700 2400 7600 2400
+Wire Wire Line
+	7600 2500 7700 2500
+Wire Wire Line
+	7700 2600 7600 2600
+Wire Wire Line
+	7600 2700 7700 2700
+Text Label 6700 2700 0    60   ~ 0
+INT_J
+Text Label 6700 2600 0    60   ~ 0
+SDA_J
+Text Label 6700 2500 0    60   ~ 0
+SCL_J
+Text Label 6700 2400 0    60   ~ 0
+VDD3V3_J
+Text Label 2800 2300 0    60   ~ 0
+VDD3V3_J
+Text Label 3800 4500 0    60   ~ 0
+VDD3V3_J
+Text Label 6600 4700 0    60   ~ 0
+SDA_J
+Text Label 6600 4600 0    60   ~ 0
+SCL_J
 $EndSCHEMATC

Commit message: add led status indicators, rotary encoder
* add led indicators for motor direction, pwm, encoder (muxed with dpad) pins
* add led indicators for power in all blocks
* split dpad into a different page
* add selectable onboard rotary encoder for testing or user input
Parts:
- added D?: Led_Small, symbol Led_Small
- added R?: 2k, symbol R_Small
Connections:
- wire segments 55 -> 43
Changed lines of the file:
@@
 $Descr A4 11693 8268
 encoding utf-8
-Sheet 5 7
+Sheet 5 8
 Title ""
 Date ""
@@
 L GND #PWR?
 U 1 1 5762DC6A
-P 3400 3000
-F 0 "#PWR?" H 3400 2750 50  0001 C CNN
-F 1 "GND" H 3400 2850 50  0000 C CNN
-F 2 "" H 3400 3000 50  0000 C CNN
-F 3 "" H 3400 3000 50  0000 C CNN
-	1    3400 3000
-	1    0    0    -1
-$EndComp
-Wire Wire Line
-	3400 3000 3400 2900
-Wire Wire Line
-	3400 2900 3500 2900
-Wire Wire Line
-	3500 2900 3900 2900
-Wire Wire Line
-	3900 2900 4300 2900
-Wire Wire Line
-	4300 2900 4700 2900
-Wire Wire Line
-	4700 2900 5000 2900
-Wire Wire Line
-	5000 2900 5100 2900
+P 3400 3200
+F 0 "#PWR?" H 3400 2950 50  0001 C CNN
+F 1 "GND" H 3400 3050 50  0000 C CNN
+F 2 "" H 3400 3200 50  0000 C CNN
+F 3 "" H 3400 3200 50  0000 C CNN
+	1    3400 3200
+	1    0    0    -1
+$EndComp
+Wire Wire Line
+	3400 3200 3400 2900
+Wire Wire Line
+	3400 2900 5100 2900
 Wire Wire Line
 	5100 2800 5000 2800
@@
 Connection ~ 3500 2900
 Wire Wire Line
-	2800 2300 3500 2300
-Wire Wire Line
-	3500 2300 3900 2300
-Wire Wire Line
-	3900 2300 4300 2300
-Wire Wire Line
-	4300 2300 5100 2300
+	2800 2300 5100 2300
 Wire Wire Line
 	3500 2300 3500 2600
@@
 Connection ~ 3900 2300
 Wire Wire Line
-	4300 2300 4300 2400
-Wire Wire Line
-	4300 2400 4300 2600
+	4300 2300 4300 2600
 Connection ~ 4300 2300
 Wire Wire Line
@@
 INT
 Wire Wire Line
-	7100 2700 6600 2700
-Wire Wire Line
-	6600 2700 6500 2700
+	6500 2700 7100 2700
 Text HLabel 7700 2500 2    60   Input ~ 0
 SCL
@@
 	6500 2500 7100 2500
 Wire Wire Line
-	6500 2400 6600 2400
-Wire Wire Line
-	6600 2400 7100 2400
+	6500 2400 7100 2400
 $Comp
 L BMP180 U?
@@
 $EndComp
 Wire Wire Line
-	3800 4500 4500 4500
-Wire Wire Line
-	4500 4500 4900 4500
-Wire Wire Line
-	4900 4500 5300 4500
+	3800 4500 5300 4500
 Wire Wire Line
 	4500 4700 4500 4500
 Connection ~ 4500 4500
 Wire Wire Line
-	4900 4700 4900 4600
-Wire Wire Line
-	4900 4600 4900 4500
+	4900 4500 4900 4700
 Connection ~ 4900 4500
 Wire Wire Line
@@
 	5200 4800 5200 5000
 Wire Wire Line
-	5200 5000 4900 5000
-Wire Wire Line
-	4900 5000 4500 5000
-Wire Wire Line
-	4500 5000 4400 5000
+	5200 5000 4400 5000
 Wire Wire Line
 	4400 5000 4400 5100
@@
 Text Label 6600 4600 0    60   ~ 0
 SCL_J
+$Comp
+L Led_Small D?
+U 1 1 5770C700
+P 3100 2600
+F 0 "D?" H 3050 2725 50  0000 L CNN
+F 1 "Led_Small" H 2925 2500 50  0000 L CNN
+F 2 "" V 3100 2600 50  0000 C CNN
+F 3 "" V 3100 2600 50  0000 C CNN
+	1    3100 2600
+	0    -1   -1   0
+$EndComp
+$Comp
+L R_Small R?
+U 1 1 5770C793
+P 3100 2900
+F 0 "R?" H 3130 2920 50  0000 L CNN
+F 1 "2k" H 3130 2860 50  0000 L CNN
+F 2 "" H 3100 2900 50  0000 C CNN
+F 3 "" H 3100 2900 50  0000 C CNN
+	1    3100 2900
+	1    0    0    -1
+$EndComp
+Wire Wire Line
+	3100 2500 3100 2300
+Connection ~ 3100 2300
+Wire Wire Line
+	3100 2700 3100 2800
+Wire Wire Line
+	3100 3000 3100 3100
+Wire Wire Line
+	3100 3100 3400 3100
+Connection ~ 3400 3100
 $EndSCHEMATC

Commit message: make extra footprints. start floorplan. fix display nets. add power expansion header.
Parts:
- C501: renamed from C?; footprint (none) -> Capacitors_Tantalum_SMD:TantalC_SizeA_EIA-3216_Wave
- C502, C503, C504, C505, C506: renamed from C?; footprint (none) -> Capacitors_SMD:C_0603
- D501: renamed from D?; footprint (none) -> LEDs:LED-0603
- R501: renamed from R?; footprint (none) -> Resistors_SMD:R_0603
- SW501: renamed from SW?; footprint (none) -> labio-special:DIP-8_W7.62mm_SMT
- U501: renamed from U?; footprint (none) -> labio-special:LSM303-LGA-12
- U502: renamed from U?; footprint (none) -> labio-special:BMP180-LGA-7
Changed lines of the file:
@@
 $Descr A4 11693 8268
 encoding utf-8
-Sheet 5 8
+Sheet 5 9
 Title ""
 Date ""
@@
 6-DOF Accelerometer + Compass\n\nKeep currents higher than 10mA\na few mm away from compass.\n\n7-bit I2C Addr:
 $Comp
-L LSM303 U?
+L LSM303 U501
 U 1 1 5762DC27
 P 5800 2600
-F 0 "U?" H 5300 3050 60  0000 L CNN
+F 0 "U501" H 5300 3050 60  0000 L CNN
 F 1 "LSM303" H 5300 2150 60  0000 L CNN
-F 2 "" H 5800 2550 60  0000 C CNN
+F 2 "labio-special:LSM303-LGA-12" H 5800 2550 60  0001 C CNN
 F 3 "" H 5800 2550 60  0000 C CNN
 	1    5800 2600
@@
 $EndComp
 $Comp
-L GND #PWR?
+L GND #PWR010
 U 1 1 5762DC6A
 P 3400 3200
-F 0 "#PWR?" H 3400 2950 50  0001 C CNN
+F 0 "#PWR010" H 3400 2950 50  0001 C CNN
 F 1 "GND" H 3400 3050 50  0000 C CNN
 F 2 "" H 3400 3200 50  0000 C CNN
@@
 Connection ~ 5000 2900
 $Comp
-L C_Small C?
+L C_Small C505
 U 1 1 5762DC8A
 P 4700 2700
-F 0 "C?" H 4710 2770 50  0000 L CNN
+F 0 "C505" H 4710 2770 50  0000 L CNN
 F 1 "0.1uF" H 4710 2620 50  0000 L CNN
-F 2 "" H 4700 2700 50  0000 C CNN
+F 2 "Capacitors_SMD:C_0603" H 4700 2700 50  0001 C CNN
 F 3 "" H 4700 2700 50  0000 C CNN
 	1    4700 2700
@@
 $EndComp
 $Comp
-L C_Small C?
+L C_Small C503
 U 1 1 5762DD09
 P 4300 2700
-F 0 "C?" H 4310 2770 50  0000 L CNN
+F 0 "C503" H 4310 2770 50  0000 L CNN
 F 1 "0.1uF" H 4310 2620 50  0000 L CNN
-F 2 "" H 4300 2700 50  0000 C CNN
+F 2 "Capacitors_SMD:C_0603" H 4300 2700 50  0001 C CNN
 F 3 "" H 4300 2700 50  0000 C CNN
 	1    4300 2700
@@
 $EndComp
 $Comp
-L C_Small C?
+L C_Small C502
 U 1 1 5762DD26
 P 3900 2700
-F 0 "C?" H 3910 2770 50  0000 L CNN
+F 0 "C502" H 3910 2770 50  0000 L CNN
 F 1 "0.1uF" H 3910 2620 50  0000 L CNN
-F 2 "" H 3900 2700 50  0000 C CNN
+F 2 "Capacitors_SMD:C_0603" H 3900 2700 50  0001 C CNN
 F 3 "" H 3900 2700 50  0000 C CNN
 	1    3900 2700
@@
 $EndComp
 $Comp
-L CP_Small C?
+L CP_Small C501
 U 1 1 5762DD77
 P 3500 2700
-F 0 "C?" H 3510 2770 50  0000 L CNN
+F 0 "C501" H 3510 2770 50  0000 L CNN
 F 1 "10uF" H 3510 2620 50  0000 L CNN
-F 2 "" H 3500 2700 50  0000 C CNN
+F 2 "Capacitors_Tantalum_SMD:TantalC_SizeA_EIA-3216_Wave" H 3500 2700 50  0001 C CNN
 F 3 "" H 3500 2700 50  0000 C CNN
 	1    3500 2700
@@
 	6500 2400 7100 2400
 $Comp
-L BMP180 U?
+L BMP180 U502
 U 1 1 576424DA
 P 5800 4700
-F 0 "U?" H 5500 5050 60  0000 L CNN
+F 0 "U502" H 5500 5050 60  0000 L CNN
 F 1 "BMP180" H 5500 4450 60  0000 L CNN
-F 2 "" H 5300 4500 60  0000 C CNN
+F 2 "labio-special:BMP180-LGA-7" H 5300 4500 60  0001 C CNN
 F 3 "" H 5300 4500 60  0000 C CNN
 	1    5800 4700
@@
 $EndComp
 $Comp
-L C_Small C?
+L C_Small C506
 U 1 1 57642543
 P 4900 4800
-F 0 "C?" H 4910 4870 50  0000 L CNN
+F 0 "C506" H 4910 4870 50  0000 L CNN
 F 1 "0.1uF" H 4910 4720 50  0000 L CNN
-F 2 "" H 4900 4800 50  0000 C CNN
+F 2 "Capacitors_SMD:C_0603" H 4900 4800 50  0001 C CNN
 F 3 "" H 4900 4800 50  0000 C CNN
 	1    4900 4800
@@
 $EndComp
 $Comp
-L C_Small C?
+L C_Small C504
 U 1 1 5764258F
 P 4500 4800
-F 0 "C?" H 4510 4870 50  0000 L CNN
+F 0 "C504" H 4510 4870 50  0000 L CNN
 F 1 "0.1uF" H 4510 4720 50  0000 L CNN
-F 2 "" H 4500 4800 50  0000 C CNN
+F 2 "Capacitors_SMD:C_0603" H 4500 4800 50  0001 C CNN
 F 3 "" H 4500 4800 50  0000 C CNN
 	1    4500 4800
@@
 Connection ~ 4900 5000
 $Comp
-L GND #PWR?
+L GND #PWR011
 U 1 1 57642751
 P 4400 5100
-F 0 "#PWR?" H 4400 4850 50  0001 C CNN
+F 0 "#PWR011" H 4400 4850 50  0001 C CNN
 F 1 "GND" H 4400 4950 50  0000 C CNN
 F 2 "" H 4400 5100 50  0000 C CNN
@@
 Connection ~ 6600 2700
 $Comp
-L DIP_SWITCH_X04 SW?
+L DIP_SWITCH_X04 SW501
 U 1 1 576D37BB
 P 7350 2550
-F 0 "SW?" H 7350 2800 50  0000 C CNN
+F 0 "SW501" H 7350 2800 50  0000 C CNN
 F 1 "DIP_SWITCH_X04" H 7350 2300 50  0000 C CNN
-F 2 "" H 7350 1350 50  0000 C CNN
+F 2 "labio-special:DIP-8_W7.62mm_SMT" H 7350 1350 50  0001 C CNN
 F 3 "" H 7350 1350 50  0000 C CNN
 	1    7350 2550
@@
 SCL_J
 $Comp
-L Led_Small D?
+L Led_Small D501
 U 1 1 5770C700
 P 3100 2600
-F 0 "D?" H 3050 2725 50  0000 L CNN
+F 0 "D501" H 3050 2725 50  0000 L CNN
 F 1 "Led_Small" H 2925 2500 50  0000 L CNN
-F 2 "" V 3100 2600 50  0000 C CNN
+F 2 "LEDs:LED-0603" V 3100 2600 50  0001 C CNN
 F 3 "" V 3100 2600 50  0000 C CNN
 	1    3100 2600
@@
 $EndComp
 $Comp
-L R_Small R?
+L R_Small R501
 U 1 1 5770C793
 P 3100 2900
-F 0 "R?" H 3130 2920 50  0000 L CNN
+F 0 "R501" H 3130 2920 50  0000 L CNN
 F 1 "2k" H 3130 2860 50  0000 L CNN
-F 2 "" H 3100 2900 50  0000 C CNN
+F 2 "Resistors_SMD:R_0603" H 3100 2900 50  0001 C CNN
 F 3 "" H 3100 2900 50  0000 C CNN
 	1    3100 2900

Commit message: floorplan on 150x85mm board, use al caps for motors
Parts:
- removed C501: 10uF, Capacitors_Tantalum_SMD:TantalC_SizeA_EIA-3216_Wave, symbol CP_Small
- added C501: 4.7uF, Capacitors_SMD:C_0603, symbol C_Small
Changed lines of the file:
@@
-	1    0    0    -1
-$EndComp
-$Comp
-L CP_Small C501
-U 1 1 5762DD77
-P 3500 2700
-F 0 "C501" H 3510 2770 50  0000 L CNN
-F 1 "10uF" H 3510 2620 50  0000 L CNN
-F 2 "Capacitors_Tantalum_SMD:TantalC_SizeA_EIA-3216_Wave" H 3500 2700 50  0001 C CNN
-F 3 "" H 3500 2700 50  0000 C CNN
-	1    3500 2700
 	1    0    0    -1
 $EndComp
@@
 	3100 3100 3400 3100
 Connection ~ 3400 3100
+$Comp
+L C_Small C501
+U 1 1 577DEFF4
+P 3500 2700
+F 0 "C501" H 3510 2770 50  0000 L CNN
+F 1 "4.7uF" H 3510 2620 50  0000 L CNN
+F 2 "Capacitors_SMD:C_0603" H 3500 2700 50  0001 C CNN
+F 3 "" H 3500 2700 50  0000 C CNN
+	1    3500 2700
+	1    0    0    -1
+$EndComp
 $EndSCHEMATC

Commit message: first pass routing, fixed audio header 3v3 net
Parts:
- C501: footprint Capacitors_SMD:C_0603 -> Capacitors_SMD:C_0805
Changed lines of the file:
@@
 F 0 "C501" H 3510 2770 50  0000 L CNN
 F 1 "4.7uF" H 3510 2620 50  0000 L CNN
-F 2 "Capacitors_SMD:C_0603" H 3500 2700 50  0001 C CNN
+F 2 "Capacitors_SMD:C_0805" H 3500 2700 50  0001 C CNN
 F 3 "" H 3500 2700 50  0000 C CNN
 	1    3500 2700
