File: pcb/labio.kicad_pcb (KiCad board)
At the start: 2 copper layers, 152 x 85 mm, 235 parts, among them IC201 dnp-AT24CS32-XHM, J701 JACK_TRRS_6PINS, P201 CONN_02X20, P301 CONN_01X04, P302 CONN_01X04, P303 CONN_01X04, P401 SFV12R-1ST__HLF, P601 CONN_01X02, P602 CONN_01X02, P603 CONN_01X04, P604 CONN_01X02, P605 CONN_01X03, P606 CONN_01X03, P607 CONN_01X05, P608 CONN_01X05, P701 CONN_01X04, P702 CONN_01X04, P703 CONN_01X04, P704 CONN_01X02, P901 CONN_01X06, Q301 PHOTOTRANSISTOR, Q302 Q_NMOS_GSD, Q303 Q_NMOS_GSD, Q601 Q_NMOS_GSD, Q602 Q_NMOS_GSD, Q603 Q_NMOS_GSD, Q604 Q_NMOS_GSD, Q605 Q_NMOS_GSD, Q606 Q_NMOS_GSD, Q607 Q_NMOS_GSD, Q608 Q_NMOS_GSD, Q609 Q_NMOS_GSD, Q610 Q_NMOS_GSD, Q611 Q_NMOS_GSD, Q612 Q_NMOS_GSD, Q613 Q_NMOS_GSD, SW301 DIP_SWITCH_X04, SW401 DIP_SWITCH_X04, SW501 DIP_SWITCH_X04, SW601 DIP_SWITCH_X04, SW602 DIP_SWITCH_X04, SW603 DIP_SWITCH_X04, SW604 DIP_SWITCH_X04, SW605 ROT_ENC, SW606 DIP_SWITCH_X04, SW701 DIP_SWITCH_X04, SW702 DIP_SWITCH_X04, SW801 SW_PUSH, SW802 SW_PUSH, SW803 SW_PUSH, SW804 SW_PUSH, SW805 SW_PUSH, U201 AP7365_SOT-23-5, U301 ADS1015, U501 LSM303D, U502 BMP280, U503 L3GD20H, U601 L298P_PowerSO20, U701 SPU0410HR5H, U702 WM8750, U703 OPA344_SOT23-5

Commit message: adjust vdd servo, vdd codec pours
Parts:
- moved D601 0.25 mm to (174.2, 119.8)
- moved R607 0.25 mm to (176.8, 119.8)
Changed lines of the file:
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@@
     (thickness 1.6)
     (drawings 178)
-    (tracks 2697)
+    (tracks 2696)
     (zones 0)
     (modules 235)
@@
   )
   (module LEDs:LED-0603 (layer F.Cu)
-    (at 174.25 120 90)
+    (at 174.25 119.75 90)
     (descr "LED 0603 smd package")
     (tags "LED led 0603 SMD smd SMT smt smdled SMDLED smtled SMTLED")
@@
   )
   (module Resistors_SMD:R_0603 (layer F.Cu)
-    (at 176.75 120 90)
+    (at 176.75 119.75 90)
     (descr "Resistor SMD 0603, reflow soldering, Vishay (see dcrcw.pdf)")
     (tags "resistor 0603")
@@
     (tags "resistor 1206")
     (attr smd)
-    (fp_text reference F604 (at 0 -1.75 180) (layer F.SilkS)
+    (fp_text reference F604 (at 2.5 0 270) (layer F.SilkS)
       (effects (font (size 0.7 0.7) (thickness 0.15)))
     )
@@
   (segment (start 220 83.25) (end 220 84) (width 0.254) (layer F.Cu) (net 1))
   (via (at 220 84) (size 0.6096) (drill 0.3048) (layers F.Cu B.Cu) (net 1))
-  (segment (start 176.75 119.25) (end 176.75 118.75) (width 0.254) (layer F.Cu) (net 1))
-  (via (at 176.75 118.75) (size 0.6096) (drill 0.3048) (layers F.Cu B.Cu) (net 1))
+  (segment (start 176.75 119) (end 176.75 118.5) (width 0.254) (layer F.Cu) (net 1))
+  (via (at 176.75 118.5) (size 0.6096) (drill 0.3048) (layers F.Cu B.Cu) (net 1))
   (segment (start 217.125 79.75) (end 217.125 79.125) (width 0.254) (layer F.Cu) (net 1))
   (segment (start 217.125 79.125) (end 216.5 78.5) (width 0.254) (layer F.Cu) (net 1))
@@
   (segment (start 93.5 58.25) (end 93.25 58) (width 0.254) (layer F.Cu) (net 3))
   (segment (start 93.25 58) (end 93.25 57) (width 0.254) (layer F.Cu) (net 3))
+  (segment (start 174.05 117.8) (end 174.25 118) (width 0.254) (layer F.Cu) (net 4))
+  (segment (start 174.25 118) (end 174.25 119.0007) (width 0.254) (layer F.Cu) (net 4))
+  (segment (start 174.05 116.5) (end 174.05 117.8) (width 0.254) (layer F.Cu) (net 4))
   (segment (start 174 114.25) (end 178.75 114.25) (width 0.254) (layer F.Cu) (net 4))
   (segment (start 178.75 114.25) (end 180.25 112.75) (width 0.254) (layer F.Cu) (net 4))
@@
   (segment (start 172.5 112.75) (end 174 114.25) (width 0.254) (layer F.Cu) (net 4))
   (segment (start 171.5 112.75) (end 172.5 112.75) (width 0.254) (layer F.Cu) (net 4))
-  (segment (start 174.05 118.05) (end 174.25 118.25) (width 0.254) (layer F.Cu) (net 4))
-  (segment (start 174.25 118.25) (end 174.25 119.2507) (width 0.254) (layer F.Cu) (net 4))
-  (segment (start 174.05 116.5) (end 174.05 118.05) (width 0.254) (layer F.Cu) (net 4))
   (segment (start 176.75 92.5) (end 179.25 92.5) (width 0.254) (layer F.Cu) (net 4))
   (segment (start 179.75 93) (end 179.445201 92.695201) (width 0.254) (layer F.Cu) (net 4))
@@
   (segment (start 81.75 78.25) (end 81.75 80.7493) (width 0.254) (layer F.Cu) (net 26))
   (segment (start 81.75 80.7493) (end 81.7493 80.75) (width 0.254) (layer F.Cu) (net 26))
-  (segment (start 176.75 120.75) (end 174.2507 120.75) (width 0.254) (layer F.Cu) (net 27))
-  (segment (start 174.2507 120.75) (end 174.25 120.7493) (width 0.254) (layer F.Cu) (net 27))
+  (segment (start 176.75 120.5) (end 174.2507 120.5) (width 0.254) (layer F.Cu) (net 27))
+  (segment (start 174.2507 120.5) (end 174.25 120.4993) (width 0.254) (layer F.Cu) (net 27))
   (segment (start 166.0507 71) (end 166.0507 73.4993) (width 0.254) (layer F.Cu) (net 28))
   (segment (start 166.0507 73.4993) (end 166.05 73.5) (width 0.254) (layer F.Cu) (net 28))
@@
   (via (at 112 97.5) (size 0.6096) (drill 0.3048) (layers F.Cu B.Cu) (net 152))
   (segment (start 100.92 93.93) (end 102.23 93.93) (width 0.254) (layer F.Cu) (net 152))
+  (segment (start 178.5 123.5) (end 178.75 123.25) (width 0.254) (layer B.Cu) (net 153))
+  (segment (start 178.75 123.25) (end 178.75 112.75) (width 0.254) (layer B.Cu) (net 153))
+  (segment (start 178.75 112.75) (end 178.5 112.5) (width 0.254) (layer B.Cu) (net 153))
+  (segment (start 178.75 123.75) (end 178.75 131.815) (width 0.254) (layer F.Cu) (net 153))
+  (segment (start 178.75 123.75) (end 178.5 123.5) (width 0.254) (layer F.Cu) (net 153))
+  (via (at 178.5 123.5) (size 0.6096) (drill 0.3048) (layers F.Cu B.Cu) (net 153))
   (segment (start 166.75 84.5) (end 166.75 88) (width 0.254) (layer B.Cu) (net 153))
   (segment (start 170.25 81) (end 166.75 84.5) (width 0.254) (layer B.Cu) (net 153))
@@
   (segment (start 136.5 95) (end 113.5 95) (width 0.254) (layer F.Cu) (net 153))
   (segment (start 136.5 95) (end 138.5 93) (width 0.254) (layer F.Cu) (net 153))
-  (segment (start 178.75 121) (end 178.75 131.815) (width 0.254) (layer F.Cu) (net 153))
-  (segment (start 178.5 120.75) (end 178.75 121) (width 0.254) (layer F.Cu) (net 153))
-  (segment (start 178.75 120.5) (end 178.5 120.75) (width 0.254) (layer B.Cu) (net 153))
-  (via (at 178.5 120.75) (size 0.6096) (drill 0.3048) (layers F.Cu B.Cu) (net 153))
-  (segment (start 178.75 112.75) (end 178.75 115.75) (width 0.254) (layer B.Cu) (net 153))
-  (segment (start 178.5 112.5) (end 178.75 112.75) (width 0.254) (layer B.Cu) (net 153))
   (segment (start 178.75 100.205638) (end 178.75 112.25) (width 0.254) (layer F.Cu) (net 153))
   (segment (start 178.75 112.25) (end 178.5 112.5) (width 0.254) (layer F.Cu) (net 153))
@@
   (segment (start 164.507036 95.242964) (end 164.507036 93.167168) (width 0.254) (layer B.Cu) (net 153))
   (segment (start 164.5 95.25) (end 164.507036 95.242964) (width 0.254) (layer B.Cu) (net 153))
-  (segment (start 178.75 115.75) (end 178.75 120.5) (width 0.254) (layer B.Cu) (net 153))
   (segment (start 178.75 131.815) (end 179.705 132.77) (width 0.254) (layer F.Cu) (net 153))
   (segment (start 170.25 80.25) (end 170.25 78.20076) (width 0.254) (layer F.Cu) (net 153))
@@
   (via (at 154.5 90) (size 0.6096) (drill 0.3048) (layers F.Cu B.Cu) (net 156))
   (segment (start 106.08 104.09) (end 104.77 104.09) (width 0.254) (layer F.Cu) (net 156))
+  (segment (start 179.5 123.5) (end 179.262008 123.262008) (width 0.254) (layer B.Cu) (net 157))
+  (segment (start 179.262008 123.262008) (end 179.262008 120.512008) (width 0.254) (layer B.Cu) (net 157))
+  (segment (start 179.262008 120.512008) (end 179.25 120.5) (width 0.254) (layer B.Cu) (net 157))
+  (segment (start 179.25 120.5) (end 179.25 112.75) (width 0.254) (layer B.Cu) (net 157))
+  (segment (start 179.25 112.75) (end 179.5 112.5) (width 0.254) (layer B.Cu) (net 157))
+  (segment (start 179.25 127.5) (end 179.25 123.75) (width 0.254) (layer F.Cu) (net 157))
+  (segment (start 179.25 123.75) (end 179.5 123.5) (width 0.254) (layer F.Cu) (net 157))
+  (via (at 179.5 123.5) (size 0.6096) (drill 0.3048) (layers F.Cu B.Cu) (net 157))
   (segment (start 170.5 84.568948) (end 170.5 89.25) (width 0.254) (layer B.Cu) (net 157))
   (segment (start 170.5 89.25) (end 169.75 90) (width 0.254) (layer B.Cu) (net 157))
@@
   (segment (start 113.25 94.5) (end 110.5 97.25) (width 0.254) (layer F.Cu) (net 157))
   (segment (start 107.22 96.47) (end 106.08 96.47) (width 0.254) (layer F.Cu) (net 157))
-  (segment (start 179.5 120.75) (end 179.25 121) (width 0.254) (layer F.Cu) (net 157))
   (segment (start 187.2474 130) (end 189.865 132.6176) (width 0.254) (layer F.Cu) (net 157))
-  (segment (start 179.25 121) (end 179.25 127.5) (width 0.254) (layer F.Cu) (net 157))
   (segment (start 181.75 130) (end 187.2474 130) (width 0.254) (layer F.Cu) (net 157))
   (segment (start 179.25 127.5) (end 181.75 130) (width 0.254) (layer F.Cu) (net 157))
   (segment (start 189.865 132.6176) (end 189.865 132.77) (width 0.254) (layer F.Cu) (net 157))
-  (segment (start 179.25 120) (end 179.25 120.5) (width 0.254) (layer B.Cu) (net 157))
-  (segment (start 179.25 120.5) (end 179.5 120.75) (width 0.254) (layer B.Cu) (net 157))
-  (via (at 179.5 120.75) (size 0.6096) (drill 0.3048) (layers F.Cu B.Cu) (net 157))
-  (segment (start 179.25 112.75) (end 179.25 115.25) (width 0.254) (layer B.Cu) (net 157))
-  (segment (start 179.5 112.5) (end 179.25 112.75) (width 0.254) (layer B.Cu) (net 157))
   (segment (start 179.25 100.059045) (end 179.25 112.25) (width 0.254) (layer F.Cu) (net 157))
   (segment (start 179.25 112.25) (end 179.5 112.5) (width 0.254) (layer F.Cu) (net 157))
@@
   (segment (start 169.5 93.194216) (end 169.507036 93.18718) (width 0.254) (layer B.Cu) (net 157))
   (via (at 169.5 95) (size 0.6096) (drill 0.3048) (layers F.Cu B.Cu) (net 157))
-  (segment (start 179.25 115.25) (end 179.25 120) (width 0.254) (layer B.Cu) (net 157))
   (segment (start 174.5 80.25) (end 174.5 78.20076) (width 0.254) (layer F.Cu) (net 157))
   (segment (start 174.5 78.20076) (end 174.3 78.00076) (width 0.254) (layer F.Cu) (net 157))
@@
     (polygon
       (pts
-        (xy 172.5 134.5) (xy 193.5 134.5) (xy 193.5 96) (xy 172.5 96)
+        (xy 170.75 134.5) (xy 193.5 134.5) (xy 193.5 96) (xy 179.5 96) (xy 179.5 114.75)
+        (xy 170.75 123.5)
       )
     )
@@
       (pts
         (xy 194 134.5) (xy 194 96) (xy 213.75 96) (xy 221 88.75) (xy 221 87)
-        (xy 215.75 87) (xy 215.75 64.75) (xy 222 64.75) (xy 222 86) (xy 228.5 86)
-        (xy 228.5 123.5) (xy 228.5 132.5) (xy 226.5 134.5)
+        (xy 215.75 87) (xy 215.75 64.75) (xy 222 64.75) (xy 222 83.25) (xy 224.75 86)
+        (xy 228.5 86) (xy 228.5 123.5) (xy 228.5 132.5) (xy 226.5 134.5)
       )
     )
