File: pcb/labio-dio.sch (KiCad schematic (older format))
At the start: 100 parts, among them P601 CONN_01X02, P602 CONN_01X02, P603 CONN_01X04, P604 CONN_01X02, P605 CONN_01X03, P606 CONN_01X03, P607 CONN_01X05, P608 CONN_01X05, Q601 Q_NMOS_GSD, Q602 Q_NMOS_GSD, Q603 Q_NMOS_GSD, Q604 Q_NMOS_GSD, Q605 Q_NMOS_GSD, Q606 Q_NMOS_GSD, Q607 Q_NMOS_GSD, Q608 Q_NMOS_GSD, Q609 Q_NMOS_GSD, Q610 Q_NMOS_GSD, Q611 Q_NMOS_GSD, Q612 Q_NMOS_GSD, Q613 Q_NMOS_GSD, SW601 DIP_SWITCH_X04, SW602 DIP_SWITCH_X04, SW603 DIP_SWITCH_X04, SW604 DIP_SWITCH_X04, SW605 ROT_ENC, SW606 DIP_SWITCH_X04, U601 L298P_PowerSO20

Commit message: add bom. change led resistors to 220 and dnp rpi hat eeprom
Parts:
- R605, R606, R607, R612, R613, R618, R619, R622, R623, R624, R626, R627, R630, R631, R634, R635: value 2k -> 220
Changed lines of the file:
@@
 P 1600 5100
 F 0 "R605" H 1630 5120 50  0000 L CNN
-F 1 "2k" H 1630 5060 50  0000 L CNN
+F 1 "220" H 1630 5060 50  0000 L CNN
 F 2 "Resistors_SMD:R_0603" H 1600 5100 50  0001 C CNN
 F 3 "" H 1600 5100 50  0000 C CNN
@@
 P 1600 6600
 F 0 "R606" H 1630 6620 50  0000 L CNN
-F 1 "2k" H 1630 6560 50  0000 L CNN
+F 1 "220" H 1630 6560 50  0000 L CNN
 F 2 "Resistors_SMD:R_0603" H 1600 6600 50  0001 C CNN
 F 3 "" H 1600 6600 50  0000 C CNN
@@
 P 3100 5100
 F 0 "R612" H 3130 5120 50  0000 L CNN
-F 1 "2k" H 3130 5060 50  0000 L CNN
+F 1 "220" H 3130 5060 50  0000 L CNN
 F 2 "Resistors_SMD:R_0603" H 3100 5100 50  0001 C CNN
 F 3 "" H 3100 5100 50  0000 C CNN
@@
 P 3100 6600
 F 0 "R613" H 3130 6620 50  0000 L CNN
-F 1 "2k" H 3130 6560 50  0000 L CNN
+F 1 "220" H 3130 6560 50  0000 L CNN
 F 2 "Resistors_SMD:R_0603" H 3100 6600 50  0001 C CNN
 F 3 "" H 3100 6600 50  0000 C CNN
@@
 P 4600 5150
 F 0 "R618" H 4630 5170 50  0000 L CNN
-F 1 "2k" H 4630 5110 50  0000 L CNN
+F 1 "220" H 4630 5110 50  0000 L CNN
 F 2 "Resistors_SMD:R_0603" H 4600 5150 50  0001 C CNN
 F 3 "" H 4600 5150 50  0000 C CNN
@@
 P 4600 6650
 F 0 "R619" H 4630 6670 50  0000 L CNN
-F 1 "2k" H 4630 6610 50  0000 L CNN
+F 1 "220" H 4630 6610 50  0000 L CNN
 F 2 "Resistors_SMD:R_0603" H 4600 6650 50  0001 C CNN
 F 3 "" H 4600 6650 50  0000 C CNN
@@
 P 6100 5100
 F 0 "R622" H 6130 5120 50  0000 L CNN
-F 1 "2k" H 6130 5060 50  0000 L CNN
+F 1 "220" H 6130 5060 50  0000 L CNN
 F 2 "Resistors_SMD:R_0603" H 6100 5100 50  0001 C CNN
 F 3 "" H 6100 5100 50  0000 C CNN
@@
 P 6100 6600
 F 0 "R623" H 6130 6620 50  0000 L CNN
-F 1 "2k" H 6130 6560 50  0000 L CNN
+F 1 "220" H 6130 6560 50  0000 L CNN
 F 2 "Resistors_SMD:R_0603" H 6100 6600 50  0001 C CNN
 F 3 "" H 6100 6600 50  0000 C CNN
@@
 P 7600 5100
 F 0 "R626" H 7630 5120 50  0000 L CNN
-F 1 "2k" H 7630 5060 50  0000 L CNN
+F 1 "220" H 7630 5060 50  0000 L CNN
 F 2 "Resistors_SMD:R_0603" H 7600 5100 50  0001 C CNN
 F 3 "" H 7600 5100 50  0000 C CNN
@@
 P 9100 5100
 F 0 "R630" H 9130 5120 50  0000 L CNN
-F 1 "2k" H 9130 5060 50  0000 L CNN
+F 1 "220" H 9130 5060 50  0000 L CNN
 F 2 "Resistors_SMD:R_0603" H 9100 5100 50  0001 C CNN
 F 3 "" H 9100 5100 50  0000 C CNN
@@
 P 10600 5100
 F 0 "R634" H 10630 5120 50  0000 L CNN
-F 1 "2k" H 10630 5060 50  0000 L CNN
+F 1 "220" H 10630 5060 50  0000 L CNN
 F 2 "Resistors_SMD:R_0603" H 10600 5100 50  0001 C CNN
 F 3 "" H 10600 5100 50  0000 C CNN
@@
 P 9100 6600
 F 0 "R631" H 9130 6620 50  0000 L CNN
-F 1 "2k" H 9130 6560 50  0000 L CNN
+F 1 "220" H 9130 6560 50  0000 L CNN
 F 2 "Resistors_SMD:R_0603" H 9100 6600 50  0001 C CNN
 F 3 "" H 9100 6600 50  0000 C CNN
@@
 P 10600 6600
 F 0 "R635" H 10630 6620 50  0000 L CNN
-F 1 "2k" H 10630 6560 50  0000 L CNN
+F 1 "220" H 10630 6560 50  0000 L CNN
 F 2 "Resistors_SMD:R_0603" H 10600 6600 50  0001 C CNN
 F 3 "" H 10600 6600 50  0000 C CNN
@@
 P 1700 1800
 F 0 "R607" H 1730 1820 50  0000 L CNN
-F 1 "2k" H 1730 1760 50  0000 L CNN
+F 1 "220" H 1730 1760 50  0000 L CNN
 F 2 "Resistors_SMD:R_0603" H 1700 1800 50  0001 C CNN
 F 3 "" H 1700 1800 50  0000 C CNN
@@
 P 6300 2300
 F 0 "R624" H 6330 2320 50  0000 L CNN
-F 1 "2k" H 6330 2260 50  0000 L CNN
+F 1 "220" H 6330 2260 50  0000 L CNN
 F 2 "Resistors_SMD:R_0603" H 6300 2300 50  0001 C CNN
 F 3 "" H 6300 2300 50  0000 C CNN
@@
 P 8400 2300
 F 0 "R627" H 8430 2320 50  0000 L CNN
-F 1 "2k" H 8430 2260 50  0000 L CNN
+F 1 "220" H 8430 2260 50  0000 L CNN
 F 2 "Resistors_SMD:R_0603" H 8400 2300 50  0001 C CNN
 F 3 "" H 8400 2300 50  0000 C CNN

Commit message: Power motor driver from 5V but with 3.3V logic. Adjust R601, R602 to prevent more than 3.3V on logic lines.
Parts:
- R601, R602: value 1k -> 10k
Connections:
- net VDD_3V3: no longer SW603.4 (4A)
- net VDD_5V: now also SW603.4 (4A)
Other:
- note added: "Pull up to max 3.3V\nto protect RPi."
Changed lines of the file:
@@
 P 1200 3300
 F 0 "R602" H 1230 3320 50  0000 L CNN
-F 1 "1k" H 1230 3260 50  0000 L CNN
+F 1 "10k" H 1230 3260 50  0000 L CNN
 F 2 "Resistors_SMD:R_0603" H 1200 3300 50  0001 C CNN
 F 3 "" H 1200 3300 50  0000 C CNN
@@
 P 900 3300
 F 0 "R601" H 930 3320 50  0000 L CNN
-F 1 "1k" H 930 3260 50  0000 L CNN
+F 1 "10k" H 930 3260 50  0000 L CNN
 F 2 "Resistors_SMD:R_0603" H 900 3300 50  0001 C CNN
 F 3 "" H 900 3300 50  0000 C CNN
@@
 	1    0    0    -1
 $EndComp
-Text HLabel 6500 3300 0    60   Input ~ 0
-VDD_3V3
 Text Label 7800 3300 2    60   ~ 0
 VDD_MOT
@@
 	7400 3200 7300 3200
 Connection ~ 7400 3100
+Text Notes 700  2950 0    60   ~ 0
+Pull up to max 3.3V\nto protect RPi.
+Text HLabel 6500 3300 0    60   Input ~ 0
+VDD_5V
 $EndSCHEMATC

Commit message: add fuses for connectable headers (adc, encoder, motors, servo, codec). GERBER/BOM UPDATES ONLY
Parts:
- added F601: F_Small, labio-special:OMNI-BLOCK_Fuse_10x5mm_Littelfuse, symbol F_Small
- added F602, F603: F_Small, Resistors_SMD:R_1206, symbol F_Small
Connections:
- net VDD_ENC: now also F603.2; no longer D624.1 (K), D625.1 (K), D626.1 (K)
- net VDD_SERVO: now also F602.2; no longer D611.1 (K), D612.1 (K), D613.1 (K)
- net VS_MOTOR: now also F601.1; no longer C602.1, U601.6 (VS)
- new net VDD_ENC_F: D624.1 (K), D625.1 (K), D626.1 (K), F603.1
- new net VDD_SERVO_F: D611.1 (K), D612.1 (K), D613.1 (K), F602.1
- new net VS_MOTOR_F: C602.1, F601.2, U601.6 (VS)
Other:
- moved on the sheet: C602
Changed lines of the file:
@@
 L C_Small C602
 U 1 1 575D116B
-P 4300 1700
-F 0 "C602" H 4310 1770 50  0000 L CNN
-F 1 "0.1uF" H 4310 1620 50  0000 L CNN
-F 2 "Capacitors_SMD:C_0603" H 4300 1700 50  0001 C CNN
-F 3 "" H 4300 1700 50  0000 C CNN
-	1    4300 1700
+P 4100 1700
+F 0 "C602" H 4110 1770 50  0000 L CNN
+F 1 "0.1uF" H 4110 1620 50  0000 L CNN
+F 2 "Capacitors_SMD:C_0603" H 4100 1700 50  0001 C CNN
+F 3 "" H 4100 1700 50  0000 C CNN
+	1    4100 1700
 	1    0    0    -1
 $EndComp
@@
 	-1   0    0    1
 $EndComp
-Text Label 7800 3000 2    60   ~ 0
+Text Label 8200 3000 2    60   ~ 0
 VDD_SERVO
 Text HLabel 6500 3200 0    60   Input ~ 0
@@
 	-1   0    0    1
 $EndComp
-Text Label 10600 3400 2    60   ~ 0
+Text Label 11100 3400 2    60   ~ 0
 VDD_ENC
 Text HLabel 9300 3600 0    60   Input ~ 0
@@
 $EndComp
 NoConn ~ 1550 7000
-Text HLabel 3900 1500 0    60   Input ~ 0
+Text HLabel 5300 1350 0    60   Input ~ 0
 VS_MOTOR
 $Comp
@@
 	6900 1600 6900 1500
 Wire Wire Line
-	7300 1600 6500 1600
-Wire Wire Line
-	7300 1300 7300 1600
-Wire Wire Line
-	7500 1300 7300 1300
-Wire Wire Line
-	7500 1400 7500 1300
+	6500 1600 7300 1600
+Wire Wire Line
+	7300 1600 7300 1300
+Wire Wire Line
+	7300 1300 7500 1300
+Wire Wire Line
+	7500 1300 7500 1400
 Connection ~ 6500 1200
 Wire Wire Line
@@
 Wire Wire Line
 	6100 1200 6900 1200
-Connection ~ 4000 1500
 Connection ~ 6500 2550
 Wire Wire Line
-	6300 2550 6500 2550
-Wire Wire Line
-	6300 2400 6300 2550
+	6500 2550 6300 2550
+Wire Wire Line
+	6300 2550 6300 2400
 Wire Wire Line
 	6300 2100 6300 2200
@@
 	9900 3500 9800 3500
 Wire Wire Line
-	10100 3400 10600 3400
+	10100 3400 10500 3400
 Wire Wire Line
 	10100 3500 10200 3500
@@
 	10300 1700 9800 1700
 Wire Wire Line
-	4300 1900 5400 1900
+	4100 1900 5400 1900
 Connection ~ 5400 1700
 Wire Wire Line
@@
 Wire Wire Line
 	9500 2800 9600 2800
-Connection ~ 4300 1500
-Wire Wire Line
-	4300 1600 4300 1500
 Connection ~ 2100 1500
 Wire Wire Line
@@
 Wire Wire Line
 	2100 1800 2100 1900
-Wire Wire Line
-	4300 1900 4300 1800
 Connection ~ 8600 2900
 Wire Wire Line
@@
 Connection ~ 4000 3100
 Wire Wire Line
-	3900 3100 4000 3100
+	4000 3100 3900 3100
 Wire Wire Line
 	4000 3000 3900 3000
@@
 Wire Wire Line
 	2400 3000 2500 3000
-Wire Wire Line
-	4000 2000 3900 2000
-Wire Wire Line
-	4000 1500 4000 2000
-Wire Wire Line
-	3900 1500 5500 1500
 Wire Wire Line
 	5400 1600 5500 1600
@@
 	7100 3100 7000 3100
 Wire Wire Line
-	7300 3000 7800 3000
+	7300 3000 7500 3000
 Wire Wire Line
 	7300 3100 7400 3100
@@
 Text HLabel 6500 3300 0    60   Input ~ 0
 VDD_5V
+$Comp
+L F_Small F601
+U 1 1 57A54BF2
+P 4400 1500
+F 0 "F601" H 4360 1560 50  0000 L CNN
+F 1 "F_Small" H 4280 1440 50  0000 L CNN
+F 2 "labio-special:OMNI-BLOCK_Fuse_10x5mm_Littelfuse" H 4400 1500 50  0001 C CNN
+F 3 "" H 4400 1500 50  0000 C CNN
+	1    4400 1500
+	-1   0    0    1
+$EndComp
+Text Label 4100 1500 2    60   ~ 0
+VS_MOTOR_F
+$Comp
+L F_Small F602
+U 1 1 57A55915
+P 7600 3000
+F 0 "F602" H 7560 3060 50  0000 L CNN
+F 1 "F_Small" H 7480 2940 50  0000 L CNN
+F 2 "Resistors_SMD:R_1206" H 7600 3000 50  0001 C CNN
+F 3 "" H 7600 3000 50  0000 C CNN
+	1    7600 3000
+	1    0    0    -1
+$EndComp
+$Comp
+L F_Small F603
+U 1 1 57A55A67
+P 10600 3400
+F 0 "F603" H 10560 3460 50  0000 L CNN
+F 1 "F_Small" H 10480 3340 50  0000 L CNN
+F 2 "Resistors_SMD:R_1206" H 10600 3400 50  0001 C CNN
+F 3 "" H 10600 3400 50  0000 C CNN
+	1    10600 3400
+	1    0    0    -1
+$EndComp
+Wire Wire Line
+	10700 3400 11100 3400
+Text Label 10500 3400 2    60   ~ 0
+VDD_ENC_F
+Wire Wire Line
+	7700 3000 8200 3000
+Text Label 7500 3000 2    60   ~ 0
+VDD_SERVO_F
+Wire Wire Line
+	5400 1500 5400 1350
+Wire Wire Line
+	5400 1350 5300 1350
+Connection ~ 5400 1500
+Wire Wire Line
+	4000 1500 4300 1500
+Wire Wire Line
+	4100 1500 4100 1600
+Wire Wire Line
+	4000 1500 4000 2000
+Wire Wire Line
+	4000 2000 3900 2000
+Connection ~ 4100 1500
+Wire Wire Line
+	4500 1500 5500 1500
+Wire Wire Line
+	4100 1800 4100 1900
 $EndSCHEMATC
